File: Conference Badge/badge.brd (EAGLE design)
At the start: 82 x 50 mm, 29 parts, among them U1 ATMEGA328, U2 TPS76633D

Commit message: Correction
Routing:
- net GND: track 223.6 -> 217.3 mm
Other:
- board text added: "DQ"
- board text added: "DS18B20"
- board text added: "ICSP"
Changed lines of the file:
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@@
 <wire x1="60.6425" y1="41.91" x2="73.3425" y2="41.91" width="0.3" layer="29"/>
 <wire x1="60.6425" y1="43.18" x2="73.3425" y2="43.18" width="0.2" layer="29"/>
-<hole x="34.925" y="47.625" drill="1.5"/>
-<hole x="35.2425" y="47.625" drill="1.5"/>
-<hole x="35.56" y="47.625" drill="1.5"/>
-<hole x="35.8775" y="47.625" drill="1.5"/>
-<hole x="36.195" y="47.625" drill="1.5"/>
-<hole x="36.5125" y="47.625" drill="1.5"/>
-<hole x="36.83" y="47.625" drill="1.5"/>
-<hole x="37.1475" y="47.625" drill="1.5"/>
-<hole x="37.465" y="47.625" drill="1.5"/>
-<hole x="37.7825" y="47.625" drill="1.5"/>
-<hole x="38.1" y="47.625" drill="1.5"/>
-<hole x="38.4175" y="47.625" drill="1.5"/>
-<hole x="38.735" y="47.625" drill="1.5"/>
-<hole x="39.0525" y="47.625" drill="1.5"/>
-<hole x="39.0525" y="47.625" drill="1.5"/>
-<hole x="39.37" y="47.625" drill="1.5"/>
-<hole x="39.6875" y="47.625" drill="1.5"/>
-<hole x="40.005" y="47.625" drill="1.5"/>
-<hole x="40.3225" y="47.625" drill="1.5"/>
-<hole x="40.64" y="47.625" drill="1.5"/>
-<hole x="40.9575" y="47.625" drill="1.5"/>
+<text x="26.035" y="9.8425" size="0.8128" layer="21">DS18B20</text>
+<text x="26.035" y="6.0325" size="0.8128" layer="21">VCC</text>
+<text x="28.8925" y="6.0325" size="0.8128" layer="21">DQ</text>
+<text x="31.115" y="6.0325" size="0.8128" layer="21">GND</text>
+<wire x1="33.02" y1="22.86" x2="37.465" y2="22.86" width="0.254" layer="21"/>
+<text x="38.735" y="19.685" size="0.8128" layer="21" rot="R90">DS18B20</text>
+<text x="50.4825" y="14.2875" size="1.4224" layer="21" rot="SR0">1</text>
+<text x="52.3875" y="11.1125" size="0.8128" layer="21" rot="R90">ICSP</text>
 </plain>
 <attributes>
@@
 <wire x1="27.305" y1="2.8575" x2="29.845" y2="2.8575" width="0.254" layer="1"/>
 <wire x1="29.845" y1="2.8575" x2="29.845" y2="5.715" width="0.254" layer="1"/>
-<wire x1="29.845" y1="5.715" x2="32.385" y2="8.255" width="0.254" layer="1"/>
 <wire x1="32.385" y1="8.255" x2="32.385" y2="11.43" width="0.254" layer="1"/>
-<wire x1="32.385" y1="11.43" x2="30.48" y2="13.335" width="0.254" layer="1"/>
 <wire x1="33.3375" y1="19.2913" x2="33.3375" y2="17.78" width="0.254" layer="1"/>
 <wire x1="33.3375" y1="17.78" x2="30.48" y2="14.9225" width="0.254" layer="1"/>
